File: efr32_feather.sch (KiCad schematic (older format))
At the start: 31 parts, among them J1 USB, J2 Battery, J3 Feather_1, J4 Feather_2, J5 DEBUG, Q1 DMG2301L, U1 EFR32BG_QFN48, U2 AP2112K-3.3, U3 MCP73831-2-OT, U4 CP2102N-A01-GQFN20, Y1 32768Hz, Y2 38.4MHz

Commit message: Reversed pin header, better antenna traces, reset button
Parts:
- removed U4: CP2102N-A01-GQFN20, Package_DFN_QFN:QFN-20-1EP_4x4mm_P0.5mm_EP2.5x2.5mm, symbol Anders_ICs:CP2102N-A01-GQFN20
- added SW1: RESET, Button_Switch_SMD:SW_SPST_B3U-1000P, symbol Switch:SW_Push
- added TP1: PF6, TestPoint:TestPoint_Pad_D1.0mm, symbol Connector:TestPoint
- added TP2: PF7, TestPoint:TestPoint_Pad_D1.0mm, symbol Connector:TestPoint
- added TP3: PA5, TestPoint:TestPoint_Pad_D1.0mm, symbol Connector:TestPoint
- added TP4: PA4, TestPoint:TestPoint_Pad_D1.0mm, symbol Connector:TestPoint
- added TP5: PA3, TestPoint:TestPoint_Pad_D1.0mm, symbol Connector:TestPoint
- added U4: CP2102N-A01-GQFN24, Package_DFN_QFN:QFN-24-1EP_4x4mm_P0.5mm_EP2.6x2.6mm, symbol Interface_USB:CP2102N-A01-GQFN24
- C9: footprint Capacitor_SMD:C_0603_1608Metric -> Capacitor_SMD:C_0402_1005Metric
- L1: footprint Inductor_SMD:L_0603_1608Metric -> Inductor_SMD:L_0402_1005Metric
Connections:
- net +3V3: now also U4.5 (VIO), U4.6 (VDD), U4.7 (REGIN)
- net D0_RX: now also U1.5 (PF4); no longer U1.29 (PA4)
- net D14_A0: now also U1.31 (PB11); no longer U1.48 (PC11)
- net D15_A1: now also U1.32 (PB12); no longer U1.47 (PC10)
- net D16_A2: now also U1.33 (PB13); no longer U1.46 (PC9)
- net D17_A3: now also U1.43 (PC6); no longer U1.45 (PC8)
- net D18_A4: now also U1.44 (PC7); no longer U1.32 (PB12)
- net D19_A5: now also U1.45 (PC8); no longer U1.31 (PB11)
- net D1_TX: now also U1.6 (PF5); no longer U1.28 (PA3)
- net D22_MISO: now also U1.48 (PC11); no longer U1.30 (PA5)
- net D23_MOSI: now also U1.47 (PC10); no longer U1.43 (PC6)
- net D24_SCK: now also U1.46 (PC9); no longer U1.44 (PC7)
- net GND: now also SW1.2, U4.2 (GND), U4.25 (GND)
- net NRESET: now also SW1.1
- net USB_D+: now also U4.3 (D+)
- net USB_D-: now also U4.4 (D-)
- net USB_RX: now also U4.20 (RXD)
- net USB_TX: now also U4.21 (TXD)
- net VBUS: now also U4.8 (VBUS)
- net at U1.7 (PF6): now also TP1.1
- net at U1.8 (PF7): now also TP2.1
- net at R5.2: now also U4.9 (~RSTb)
- new net: TP5.1, U1.28 (PA3)
- new net: TP4.1, U1.29 (PA4)
- new net: TP3.1, U1.30 (PA5)
- no-connect marks 12 -> 15
Changed lines of the file:
@@
 EESchema Schematic File Version 4
-LIBS:feather-cache
+LIBS:efr32_feather-cache
 EELAYER 29 0
 EELAYER END
@@
 encoding utf-8
 Sheet 1 1
-Title ""
-Date ""
-Rev ""
+Title "EFR32 Feather"
+Date "2019-06-05"
+Rev "0.1"
 Comp ""
 Comment1 ""
@@
 	6925 3825 6675 3825
 Wire Wire Line
-	7725 2225 7725 1975
-Wire Wire Line
-	7625 2225 7625 1975
-Wire Wire Line
-	7525 2225 7525 1975
-Wire Wire Line
-	7425 2225 7425 1975
+	7925 2225 7925 1975
+Wire Wire Line
+	9025 3025 9275 3025
+Wire Wire Line
+	9025 3125 9275 3125
+Wire Wire Line
+	9025 3225 9275 3225
 Text Label 6675 3825 2    50   ~ 0
 NRESET
@@
 	1    0    0    -1
 $EndComp
-Text Label 7725 1975 1    50   ~ 0
+Text Label 7925 1975 1    50   ~ 0
 D17_A3
-Text Label 7625 1975 1    50   ~ 0
+Text Label 9275 3025 0    50   ~ 0
 D16_A2
-Text Label 7525 1975 1    50   ~ 0
+Text Label 9275 3125 0    50   ~ 0
 D15_A1
-Text Label 7425 1975 1    50   ~ 0
+Text Label 9275 3225 0    50   ~ 0
 D14_A0
 $Comp
@@
 SWDIO
 NoConn ~ 1225 1175
-Text Label 9275 3325 0    50   ~ 0
+Text Label 7425 1975 1    50   ~ 0
 D22_MISO
-Text Label 7925 1975 1    50   ~ 0
+Text Label 7525 1975 1    50   ~ 0
 D23_MOSI
+Text Label 7625 1975 1    50   ~ 0
+D24_SCK
+Text Label 7725 1975 1    50   ~ 0
+D19_A5
 Text Label 7825 1975 1    50   ~ 0
-D24_SCK
-Text Label 9275 3225 0    50   ~ 0
-D19_A5
-Text Label 9275 3125 0    50   ~ 0
 D18_A4
 Wire Wire Line
-	9025 3325 9275 3325
-Wire Wire Line
-	7925 2225 7925 1975
+	7425 2225 7425 1975
+Wire Wire Line
+	7525 2225 7525 1975
+Wire Wire Line
+	7625 2225 7625 1975
+Wire Wire Line
+	7725 2225 7725 1975
 Wire Wire Line
 	7825 2225 7825 1975
-Wire Wire Line
-	9025 3225 9275 3225
-Wire Wire Line
-	9025 3125 9275 3125
 $Comp
 L Device:Crystal_Small Y1
@@
 SWDIO
 Wire Wire Line
-	9025 3525 9275 3525
-Wire Wire Line
-	9025 3425 9275 3425
-Text Label 9275 3425 0    50   ~ 0
+	6925 3125 6675 3125
+Wire Wire Line
+	6925 3225 6675 3225
+Text Label 6675 3125 2    50   ~ 0
 D0_RX
-Text Label 9275 3525 0    50   ~ 0
+Text Label 6675 3225 2    50   ~ 0
 D1_TX
 Text Label 9275 3625 0    50   ~ 0
@@
 F 0 "L1" V 7110 4825 50  0000 C CNN
 F 1 "1.9nH" V 7019 4825 50  0000 C CNN
-F 2 "Inductor_SMD:L_0603_1608Metric" H 6925 4825 50  0001 C CNN
+F 2 "Inductor_SMD:L_0402_1005Metric" H 6925 4825 50  0001 C CNN
 F 3 "~" H 6925 4825 50  0001 C CNN
 	1    6925 4825
@@
 F 0 "C9" H 6700 5075 50  0000 L CNN
 F 1 "1.5pF" H 6700 4925 50  0000 L CNN
-F 2 "Capacitor_SMD:C_0603_1608Metric" H 6700 5000 50  0001 C CNN
+F 2 "Capacitor_SMD:C_0402_1005Metric" H 6700 5000 50  0001 C CNN
 F 3 "~" H 6700 5000 50  0001 C CNN
 	1    6700 5000
@@
 NoConn ~ 3500 4700
 $Comp
-L Anders_ICs:CP2102N-A01-GQFN20 U4
-U 1 1 5CFBDE61
-P 2900 4100
-F 0 "U4" H 2975 5025 50  0000 C CNN
-F 1 "CP2102N-A01-GQFN20" H 3375 4925 50  0000 C CNN
-F 2 "Package_DFN_QFN:QFN-20-1EP_4x4mm_P0.5mm_EP2.5x2.5mm" H 3350 3300 50  0001 L CNN
-F 3 "https://www.silabs.com/documents/public/data-sheets/cp2102n-datasheet.pdf" H 2950 3050 50  0001 C CNN
-	1    2900 4100
-	1    0    0    -1
-$EndComp
-$Comp
 L power:+3.3V #PWR0124
 U 1 1 5CFC102A
@@
 	1925 2975 1925 4100
 Connection ~ 2125 2975
-NoConn ~ 2300 3700
 NoConn ~ 2300 3800
 NoConn ~ 2300 3900
@@
 Text Notes 2900 2925 0    50   ~ 0
 USB UART
+$Comp
+L Switch:SW_Push SW1
+U 1 1 5CF736DB
+P 5850 1500
+F 0 "SW1" H 5850 1785 50  0000 C CNN
+F 1 "RESET" H 5850 1694 50  0000 C CNN
+F 2 "Button_Switch_SMD:SW_SPST_B3U-1000P" H 5850 1700 50  0001 C CNN
+F 3 "~" H 5850 1700 50  0001 C CNN
+	1    5850 1500
+	1    0    0    -1
+$EndComp
+Wire Wire Line
+	5650 1500 5400 1500
+Text Label 5400 1500 2    50   ~ 0
+NRESET
+$Comp
+L power:GND #PWR0125
+U 1 1 5CF80DD4
+P 6250 1650
+F 0 "#PWR0125" H 6250 1400 50  0001 C CNN
+F 1 "GND" H 6255 1477 50  0000 C CNN
+F 2 "" H 6250 1650 50  0001 C CNN
+F 3 "" H 6250 1650 50  0001 C CNN
+	1    6250 1650
+	1    0    0    -1
+$EndComp
+Wire Wire Line
+	6050 1500 6250 1500
+Wire Wire Line
+	6250 1500 6250 1650
+$Comp
+L Connector:TestPoint TP1
+U 1 1 5CFB6ACB
+P 6675 3325
+F 0 "TP1" V 6700 3350 50  0000 C CNN
+F 1 "PF6" V 6700 3575 50  0000 C CNN
+F 2 "TestPoint:TestPoint_Pad_D1.0mm" H 6875 3325 50  0001 C CNN
+F 3 "~" H 6875 3325 50  0001 C CNN
+	1    6675 3325
+	0    -1   -1   0
+$EndComp
+$Comp
+L Connector:TestPoint TP2
+U 1 1 5CFB7ECE
+P 6675 3425
+F 0 "TP2" V 6700 3450 50  0000 C CNN
+F 1 "PF7" V 6700 3675 50  0000 C CNN
+F 2 "TestPoint:TestPoint_Pad_D1.0mm" H 6875 3425 50  0001 C CNN
+F 3 "~" H 6875 3425 50  0001 C CNN
+	1    6675 3425
+	0    -1   -1   0
+$EndComp
+Wire Wire Line
+	6925 3425 6675 3425
+Wire Wire Line
+	6925 3325 6675 3325
+$Comp
+L Interface_USB:CP2102N-A01-GQFN24 U4
+U 1 1 5D094E59
+P 2900 4100
+F 0 "U4" H 2625 3250 50  0000 C CNN
+F 1 "CP2102N-A01-GQFN24" H 3500 3250 50  0000 C CNN
+F 2 "Package_DFN_QFN:QFN-24-1EP_4x4mm_P0.5mm_EP2.6x2.6mm" H 3350 3300 50  0001 L CNN
+F 3 "https://www.silabs.com/documents/public/data-sheets/cp2102n-datasheet.pdf" H 2950 3050 50  0001 C CNN
+	1    2900 4100
+	1    0    0    -1
+$EndComp
+NoConn ~ 3500 4000
+NoConn ~ 3500 4100
+NoConn ~ 3500 4200
+NoConn ~ 3500 3500
+Wire Wire Line
+	2900 3200 2900 2975
+Wire Wire Line
+	2900 2975 2800 2975
+Wire Wire Line
+	9025 3325 9275 3325
+Wire Wire Line
+	9025 3425 9275 3425
+Wire Wire Line
+	9025 3525 9275 3525
+$Comp
+L Connector:TestPoint TP3
+U 1 1 5D10F8A7
+P 9275 3325
+F 0 "TP3" V 9250 3250 50  0000 L CNN
+F 1 "PA5" V 9250 3500 50  0000 L CNN
+F 2 "TestPoint:TestPoint_Pad_D1.0mm" H 9475 3325 50  0001 C CNN
+F 3 "~" H 9475 3325 50  0001 C CNN
+	1    9275 3325
+	0    1    1    0
+$EndComp
+$Comp
+L Connector:TestPoint TP4
+U 1 1 5D10FBDD
+P 9275 3425
+F 0 "TP4" V 9250 3350 50  0000 L CNN
+F 1 "PA4" V 9250 3600 50  0000 L CNN
+F 2 "TestPoint:TestPoint_Pad_D1.0mm" H 9475 3425 50  0001 C CNN
+F 3 "~" H 9475 3425 50  0001 C CNN
+	1    9275 3425
+	0    1    1    0
+$EndComp
+$Comp
+L Connector:TestPoint TP5
+U 1 1 5D10FFE8
+P 9275 3525
+F 0 "TP5" V 9250 3450 50  0000 L CNN
+F 1 "PA3" V 9250 3700 50  0000 L CNN
+F 2 "TestPoint:TestPoint_Pad_D1.0mm" H 9475 3525 50  0001 C CNN
+F 3 "~" H 9475 3525 50  0001 C CNN
+	1    9275 3525
+	0    1    1    0
+$EndComp
 $EndSCHEMATC

Commit message: r0.2: moved antenna matching components, more silk screen
Parts:
- U1: symbol Anders_SiLabs_EFR32:EFR32BG_QFN48 -> efr32_feather-rescue:EFR32BG_QFN48-Anders_SiLabs_EFR32
Changed lines of the file:
@@
 Sheet 1 1
 Title "EFR32 Feather"
-Date "2019-06-05"
-Rev "0.1"
+Date "2019-06-06"
+Rev "0.2"
 Comp ""
 Comment1 ""
@@
 D14_A0
 $Comp
-L Anders_SiLabs_EFR32:EFR32BG_QFN48 U1
+L efr32_feather-rescue:EFR32BG_QFN48-Anders_SiLabs_EFR32 U1
 U 1 1 5CECF271
 P 7975 3275

Commit message: Add ESD protection for USB
Parts:
- added U1: TPD2EUSB30, Package_TO_SOT_SMD:Texas_DRT-3, symbol Power_Protection:TPD2EUSB30
- U5: renamed from U1; symbol efr32_feather-rescue:EFR32BG_QFN48-Anders_SiLabs_EFR32 -> efr32_feather-rescue:EFR32BG_QFN48-Anders_SiLabs_EFR32-efr32_feather-rescue
- renumbered C6 to C1, C7 to C2, C8 to C3, C9 to C5, C5 to C6, C1 to C7, C3 to C8, C2 to C9, D2 to D1, D1 to D2, J3 to J1, J1 to J2, J2 to J3, R2 to R1, R1 to R2, R5 to R3, R3 to R5, U4 to U3, U3 to U4, Y2 to Y1, Y1 to Y2
Connections:
- net GND: now also U1.3 (GND)
- net USB_D+: now also U1.1 (D+)
- net USB_D-: now also U1.2 (D-)
Other:
- note added: "ESD PROTECTION"
- moved on the sheet: AE1, C4, C5, C6, C7, C8, C9, J1, J2, J3, J4, J5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
